File: Board/Brytec_InputModuleRev2/Connectors.kicad_sch (KiCad schematic)
At the start: 0 parts

Commit message: Updated board
Parts:
- added J3: 6437288-2, MyKiCadLibraries:TE_6437288-2, symbol MyLibrary:6437288-2
Connections:
- net +5V: now also J3.5
- net Can1+: now also J3.4
- net Can1-: now also J3.3
- net Can2+: now also J3.2
- net Can2-: now also J3.1
- net GND: now also J3.13, J3.33
- net Ignition: now also J3.34
- net Input1: now also J3.27
- net Input10: now also J3.20
- net Input11: now also J3.19
- net Input12: now also J3.18
- net Input13: now also J3.12
- net Input14: now also J3.11
- net Input15: now also J3.10
- net Input2: now also J3.28
- net Input3: now also J3.29
- net Input4: now also J3.21
- net Input5: now also J3.30
- net Input6: now also J3.22
- net Input7: now also J3.31
- net Input8: now also J3.32
- net Input9: now also J3.26
- new net Out10: J3.16
- new net Out11: J3.17
- new net Out12: J3.23
- new net Out2: J3.24
- new net Out3: J3.9
- new net Out4: J3.8
- new net Out5: J3.6
- new net Out6: J3.15
- new net Out7: J3.14
- new net Out8: J3.25
- new net Out9: J3.7
