File: Board/Brytec_InputModuleRev2/L9966.kicad_sch (KiCad schematic)
At the start: 32 parts, among them U2 L9966CB-TR

Commit message: Updated board
Connections:
- net +12V renamed Ignition
- net SPI1_Miso renamed SPI2_Miso
- net SPI1_Mosi renamed SPI2_Mosi
- net SPI1_SS_L9966 renamed SPI2_SS_L9966
- net SPI1_Sclk renamed SPI2_Sclk
Changed lines of the file:
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@@
-    )
-  )
-  (global_label "SPI1_Sclk" (shape input) (at 167.64 99.06 0) (fields_autoplaced)
-    (effects (font (size 1.27 1.27)) (justify left))
-    (property "Intersheetrefs" "${INTERSHEET_REFS}" (at 179.7986 99.06 0)
-      (effects (font (size 1.27 1.27)) (justify left) hide)
     )
   )
@@
     )
   )
+  (global_label "Ignition" (shape input) (at 33.02 90.17 90) (fields_autoplaced)
+    (effects (font (size 1.27 1.27)) (justify left))
+    (property "Intersheetrefs" "${INTERSHEET_REFS}" (at 33.02 80.1281 90)
+      (effects (font (size 1.27 1.27)) (justify left) hide)
+    )
+  )
+  (global_label "Ignition" (shape input) (at 259.08 62.23 90) (fields_autoplaced)
+    (effects (font (size 1.27 1.27)) (justify left))
+    (property "Intersheetrefs" "${INTERSHEET_REFS}" (at 259.08 52.1881 90)
+      (effects (font (size 1.27 1.27)) (justify left) hide)
+    )
+  )
   (global_label "Input12" (shape input) (at 58.42 111.76 180) (fields_autoplaced)
     (effects (font (size 1.27 1.27)) (justify right))
@@
     )
   )
-  (global_label "SPI1_Miso" (shape input) (at 167.64 106.68 0) (fields_autoplaced)
-    (effects (font (size 1.27 1.27)) (justify left))
-    (property "Intersheetrefs" "${INTERSHEET_REFS}" (at 180.0405 106.68 0)
-      (effects (font (size 1.27 1.27)) (justify left) hide)
-    )
-  )
-  (global_label "SPI1_Mosi" (shape input) (at 167.64 104.14 0) (fields_autoplaced)
-    (effects (font (size 1.27 1.27)) (justify left))
-    (property "Intersheetrefs" "${INTERSHEET_REFS}" (at 180.0405 104.14 0)
-      (effects (font (size 1.27 1.27)) (justify left) hide)
-    )
-  )
   (global_label "Input3" (shape input) (at 218.44 76.2 0) (fields_autoplaced)
     (effects (font (size 1.27 1.27)) (justify left))
@@
     )
   )
+  (global_label "SPI2_Sclk" (shape input) (at 167.64 99.06 0) (fields_autoplaced)
+    (effects (font (size 1.27 1.27)) (justify left))
+    (property "Intersheetrefs" "${INTERSHEET_REFS}" (at 179.7986 99.06 0)
+      (effects (font (size 1.27 1.27)) (justify left) hide)
+    )
+  )
   (global_label "Input5" (shape input) (at 218.44 81.28 0) (fields_autoplaced)
     (effects (font (size 1.27 1.27)) (justify left))
@@
     )
   )
-  (global_label "SPI1_SS_L9966" (shape input) (at 167.64 101.6 0) (fields_autoplaced)
+  (global_label "SPI2_SS_L9966" (shape input) (at 167.64 101.6 0) (fields_autoplaced)
     (effects (font (size 1.27 1.27)) (justify left))
     (property "Intersheetrefs" "${INTERSHEET_REFS}" (at 185.0599 101.6 0)
@@
     )
   )
+  (global_label "SPI2_Miso" (shape input) (at 167.64 106.68 0) (fields_autoplaced)
+    (effects (font (size 1.27 1.27)) (justify left))
+    (property "Intersheetrefs" "${INTERSHEET_REFS}" (at 180.0405 106.68 0)
+      (effects (font (size 1.27 1.27)) (justify left) hide)
+    )
+  )
+  (global_label "SPI2_Mosi" (shape input) (at 167.64 104.14 0) (fields_autoplaced)
+    (effects (font (size 1.27 1.27)) (justify left))
+    (property "Intersheetrefs" "${INTERSHEET_REFS}" (at 180.0405 104.14 0)
+      (effects (font (size 1.27 1.27)) (justify left) hide)
+    )
+  )
   (global_label "Input7" (shape input) (at 218.44 86.36 0) (fields_autoplaced)
     (effects (font (size 1.27 1.27)) (justify left))
@@
     )
   )
-  (symbol (lib_id "power:+12V") (at 259.08 62.23 0) (unit 1)
-    (in_bom yes) (on_board yes) (dnp no) (fields_autoplaced)
-    (property "Reference" "#PWR012" (at 259.08 66.04 0)
-      (effects (font (size 1.27 1.27)) hide)
-    )
-    (property "Value" "+12V" (at 259.08 58.42 0)
-      (effects (font (size 1.27 1.27)))
-    )
-    (property "Footprint" "" (at 259.08 62.23 0)
-      (effects (font (size 1.27 1.27)) hide)
-    )
-    (property "Datasheet" "" (at 259.08 62.23 0)
-      (effects (font (size 1.27 1.27)) hide)
-    )
-    (pin "1")
-    (instances
-      (project "Power Module Rev 5"
-        (path "/678ed6a7-73b5-414a-90da-5837647f5dd4/405114dd-d4fe-4839-9cad-0a144ad10c54"
-          (reference "#PWR012") (unit 1)
-        )
-      )
-      (project "Brytec_InputModuleRev2"
-        (path "/864fef88-c423-4aec-8cdb-64a78dd6f95c/08375bf5-7139-4efa-85e3-4c45461a371d"
-          (reference "#PWR031") (unit 1)
-        )
-      )
-    )
-  )
   (symbol (lib_id "Device:C_Small") (at 209.55 93.98 0) (unit 1)
     (in_bom yes) (on_board yes) (dnp no)
@@
         )
       )
-    )
-  )
-  (symbol (lib_id "power:+12V") (at 33.02 90.17 0) (unit 1)
-    (in_bom yes) (on_board yes) (dnp no) (fields_autoplaced)
-    (property "Reference" "#PWR057" (at 33.02 93.98 0)
-      (effects (font (size 1.27 1.27)) hide)
-    )
-    (property "Value" "+12V" (at 33.02 86.36 0)
-      (effects (font (size 1.27 1.27)))
-    )
-    (property "Footprint" "" (at 33.02 90.17 0)
-      (effects (font (size 1.27 1.27)) hide)
-    )
-    (property "Datasheet" "" (at 33.02 90.17 0)
-      (effects (font (size 1.27 1.27)) hide)
-    )
-    (pin "1")
-    (instances
-      (project "Power Module Rev 5"
-        (path "/678ed6a7-73b5-414a-90da-5837647f5dd4/405114dd-d4fe-4839-9cad-0a144ad10c54"
-          (reference "#PWR057") (unit 1)
-        )
-      )
-      (project "Brytec_InputModuleRev2"
-        (path "/864fef88-c423-4aec-8cdb-64a78dd6f95c/08375bf5-7139-4efa-85e3-4c45461a371d"
-          (reference "#PWR022") (unit 1)
-        )
-      )
