File: Board/Brytec_InputModuleRev2/Mcu.kicad_sch (KiCad schematic)
At the start: 26 parts, among them J4 Conn_ARM_SWD_TagConnect_TC203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, J4 USB_C_Receptacle_USB2.0, U17 STM32G491CEUx, U6 MB85RS64, Y2 32.768kHz, Y3 8MHz

Commit message: Updated board
Parts:
- added R1: 0, Resistor_SMD:R_0603_1608Metric_Pad0.98x0.95mm_HandSolder, symbol Device:R_Small
Connections:
- net Can1Rx: now also U17.46 (PB8), R1.1
- net Can1Silent: now also U17.2 (PC13)
- net Can1Tx: now also U17.47 (PB9)
- net Can2Rx: now also U17.43 (PB5)
- net Can2Silent: now also U17.45 (PB7)
- net Can2Tx: now also U17.44 (PB6)
- net L6699-Int: now also U17.32 (PA10); no longer U17.42 (PB4)
- net L6699-Rst: now also U17.29 (PC6); no longer U17.40 (PC11)
- net L6699-Sync: now also U17.31 (PA9); no longer U17.45 (PB7)
- net Memory_Hold: now also U17.10 (PA2); no longer U17.12 (PA4)
- net Memory_Wp: now also U17.11 (PA3); no longer U17.17 (PB0)
- net PowerSwitchStatus: now also U17.9 (PA1); no longer U17.19 (PB2)
- net User_Led: now also U17.38 (PA15); no longer U17.22 (PB10)
- net SPI2_Sclk: now reaches U17.26 (PB13)
- net SPI2_Miso: now reaches U17.27 (PB14)
- net SPI2_Mosi: now reaches U17.28 (PB15)
- net SPI2_SS_L9966: now reaches U17.30 (PA8)
- net TLE94112_EN: now reaches U17.8 (PA0)
- net BOOT_0: no longer names the net of R1.1, S2.1
- net BOOT_0: now also R1.2; no longer U17.46 (PB8)
- net SPI1_SS_L9966: no longer names the net of U17.39 (PC10)
- net SPI1_SS_Memory: no longer names the net of U17.16 (PC4)
- net SPI1_SS_Memory: no longer U6.1 (~{CS})
- new net SPI1_SS: U17.12 (PA4), U6.1 (~{CS})
- new net SPI2_SS_TLE94112: U17.42 (PB4)
Other:
- note added: "BOOT_0"
- moved on the sheet: D2, R1
