File: Board/Brytec_InputModuleRev2/Brytec_InputModuleRev2.kicad_pcb (KiCad board)
At the start: 4 copper layers, 88.9 x 44.5 mm, 85 parts, among them J1 Conn_ARM_SWD_TagConnect_TC203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, J2 USB_C_Receptacle_USB2.0, J3 6437288-2, U1 STM32G491CEUx, U2 MB85RS64, U3 L9966CB-TR, U4 MCP2558FD-xMF, U5 MCP2558FD-xMF, U6 LMR50410Y5FQDBVRQ1, U7 TPS2116DRLR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

Commit message: Board Files
Parts:
- added G***: LOGO, Bryan_Lib:Brytec_Logo, B.Cu at (145.2, 101.7)
Other:
- board text added: "Input Module - Rev 2 2023"
